File: hardware/velocist/2Seguidor Linea.kicad_pcb (KiCad board)
At the start: 2 copper layers, 100 x 158.4 mm, 19 parts, among them J1 XT30, J2 Cable_PAD, J3 Cable_PAD, J4 QTR8a, SW1 SW_Push, SW3 SW_SPDT, U1 TB6612FNG, U2 Mini360, U3 ESP32_DEVKITC

Commit message: act pcb
Other:
- board size 100 x 158.4 mm -> 140 x 158.4 mm
Changed lines of the file:
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@@
+	)
+	(gr_line
+		(start 188.48 128.8)
+		(end 171.04 125.11)
+		(stroke
+			(width 0.05)
+			(type default)
+		)
+		(layer "Edge.Cuts")
 	)
 	(gr_line
@@
 	)
 	(gr_line
+		(start 48.47 149.45)
+		(end 48.47 184.45)
+		(stroke
+			(width 0.05)
+			(type default)
+		)
+		(layer "Edge.Cuts")
+	)
+	(gr_line
 		(start 98.47 184.45)
 		(end 48.47 184.45)
@@
 		(stroke
 			(width 0.05)
+			(type default)
+		)
+		(layer "Edge.Cuts")
+	)
+	(gr_line
+		(start 171.04 125.11)
+		(end 146.685 149.125)
+		(stroke
+			(width 0.05)

Commit message: act placa
Parts:
- moved Pololu_Micro_Gear_Motor 20.5 mm to (136.0, 167.4)
- moved Pololu_Micro_Gear_Motor 19.8 mm to (61.0, 167.3)
Routing:
- removed copper zone on B.Cu, net GND
Other:
- board size 140 x 158.4 mm -> 120 x 160 mm
Changed lines of the file:
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@@
 	(footprint "Bracket:Pololu_Micro_Bracket_Wheel_42mm"
 		(layer "F.Cu")
-		(at 115.54 167.41 -90)
+		(at 136 167.41 -90)
 		(descr "Pololu Micro Gear Motor W/Mount")
 		(property "Reference" "Pololu_Micro_Gear_Motor"
@@
 	(footprint "Bracket:Pololu_Micro_Bracket_Wheel_42mm"
 		(layer "F.Cu")
-		(at 80.83 167.41 90)
+		(at 61 167.35 90)
 		(descr "Pololu Micro Gear Motor W/Mount")
 		(property "Reference" "Pololu_Micro_Gear_Motor"
@@
 	)
 	(gr_rect
-		(start 61.66 157.87)
-		(end 126.66 175.87)
+		(start 66 157.8)
+		(end 131 175.8)
 		(stroke
 			(width 0.2)
@@
 	)
 	(gr_line
-		(start 132 43)
-		(end 132 26)
+		(start 48.5 148.9)
+		(end 48.5 103.9)
 		(stroke
 			(width 0.05)
@@
 	)
 	(gr_line
-		(start 98.5 26)
-		(end 65 26)
+		(start 158.5 188.9)
+		(end 158.5 148.9)
 		(stroke
 			(width 0.05)
@@
 	)
 	(gr_line
-		(start 107.97 43)
-		(end 132 43)
+		(start 38.5 188.9)
+		(end 38.5 148.9)
 		(stroke
 			(width 0.05)
@@
 	)
 	(gr_line
-		(start 52.04 108.8)
-		(end 52.04 148.8)
+		(start 148.5 148.9)
+		(end 148.5 103.9)
 		(stroke
 			(width 0.05)
@@
 	)
 	(gr_line
-		(start 148.47 184.45)
-		(end 148.47 149.45)
+		(start 38.5 148.9)
+		(end 48.5 148.9)
 		(stroke
 			(width 0.05)
@@
 	)
 	(gr_line
-		(start 52.04 148.8)
-		(end 48.47 149.45)
+		(start 158.5 148.9)
+		(end 148.5 148.9)
 		(stroke
 			(width 0.05)
@@
 	)
 	(gr_line
-		(start 144.9 148.8)
-		(end 148.47 149.45)
+		(start 38.5 188.9)
+		(end 158.5 188.9)
 		(stroke
 			(width 0.05)
@@
 	)
 	(gr_line
-		(start 144.9 108.8)
-		(end 144.9 148.8)
+		(start 83.4 28.9)
+		(end 113.6 28.9)
 		(stroke
 			(width 0.05)
@@
 	)
 	(gr_line
-		(start 188.48 128.8)
-		(end 171.04 125.11)
+		(start 148.5 103.9)
+		(end 130.8 86.2)
 		(stroke
 			(width 0.05)
@@
 	)
 	(gr_line
-		(start 107.97 43)
-		(end 108 83)
+		(start 98.5 28.9)
+		(end 98.5 188.9)
 		(stroke
 			(width 0.05)
@@
 	)
 	(gr_line
-		(start 89.03 43)
-		(end 65 43)
+		(start 66.2 86.2)
+		(end 130.8 86.2)
 		(stroke
 			(width 0.05)
@@
 	)
 	(gr_line
-		(start 108 83)
-		(end 144.9 108.8)
-		(stroke
-			(width 0.05)
-			(type default)
-		)
-		(layer "Edge.Cuts")
-	)
-	(gr_line
-		(start 48.47 149.45)
-		(end 48.47 184.45)
-		(stroke
-			(width 0.05)
-			(type default)
-		)
-		(layer "Edge.Cuts")
-	)
-	(gr_line
-		(start 98.47 184.45)
-		(end 48.47 184.45)
-		(stroke
-			(width 0.05)
-			(type default)
-		)
-		(layer "Edge.Cuts")
-	)
-	(gr_line
-		(start 98.47 184.45)
-		(end 148.47 184.45)
-		(stroke
-			(width 0.05)
-			(type default)
-		)
-		(layer "Edge.Cuts")
-	)
-	(gr_line
-		(start 171.04 125.11)
-		(end 146.685 149.125)
-		(stroke
-			(width 0.05)
-			(type default)
-		)
-		(layer "Edge.Cuts")
-	)
-	(gr_line
-		(start 48.47 184.45)
-		(end 48.47 149.45)
-		(stroke
-			(width 0.05)
-			(type default)
-		)
-		(layer "Edge.Cuts")
-	)
-	(gr_line
-		(start 98.5 26)
-		(end 132 26)
-		(stroke
-			(width 0.05)
-			(type default)
-		)
-		(layer "Edge.Cuts")
-	)
-	(gr_line
-		(start 89.03 43)
-		(end 89.1 83)
-		(stroke
-			(width 0.05)
-			(type default)
-		)
-		(layer "Edge.Cuts")
-	)
-	(gr_line
-		(start 65 43)
-		(end 65 26)
-		(stroke
-			(width 0.05)
-			(type default)
-		)
-		(layer "Edge.Cuts")
-	)
-	(gr_line
-		(start 89.1 83)
-		(end 52.04 108.8)
+		(start 48.5 103.9)
+		(end 66.2 86.2)
 		(stroke
 			(width 0.05)
@@
 		(net 42)
 	)
-	(zone
-		(net 6)
-		(net_name "GND")
-		(layer "B.Cu")
-		(hatch edge 0.5)
-		(connect_pads
-			(clearance 0.5)
-		)
-		(min_thickness 0.25)
-		(filled_areas_thickness no)
-		(fill yes
-			(thermal_gap 0.5)
-			(thermal_bridge_width 0.5)
-		)
-		(polygon
-			(pts
-				(xy 132 26) (xy 132 43) (xy 107.97 43) (xy 108 83) (xy 144.9 108.8) (xy 144.9 148.8) (xy 148.47 149.45)
-				(xy 148.47 184.45) (xy 48.47 184.45) (xy 48.47 149.45) (xy 52.04 148.8) (xy 52.04 108.8) (xy 89.1 83)
-				(xy 89.03 43) (xy 65 43) (xy 65 26)
-			)
-		)
-	)
 	(embedded_fonts no)

Commit message: act readme y placa
Parts:
- removed C1, C2: 104, Capacitor_THT:C_Disc_D5.0mm_W2.5mm_P2.50mm
- moved Tornillo_M3_8mm 56.2 mm to (129.4, 91.4)
- moved Tornillo_M3_8mm 55.1 mm to (69.3, 90.5)
- moved D2 40.2 mm to (61.4, 107.0), turned to 0 degrees
- moved J4 36.2 mm to (108.2, 71.7)
- moved R2 30.5 mm to (61.4, 114.5), turned to -90 degrees
- moved U2 29.6 mm to (80.0, 140.4)
- moved D1 28.7 mm to (135.6, 107.0), turned to 180 degrees
- moved R1 20.6 mm to (135.6, 114.5), turned to 90 degrees
- moved J1 15.2 mm to (135.4, 134.7), turned to 90 degrees
- moved SW3 14.9 mm to (118.2, 140.1)
- moved SW1 11.5 mm to (61.4, 131.4)
- moved U1 8.55 mm to (98.5, 140.4)
- moved U3 0.30 mm to (98.5, 111.9)
Routing:
- net +3.3V: track 105.3 -> 7.68 mm, vias 2 -> 0
- net A8: track 71.3 -> 1.75 mm
- net A7: track 70.5 -> 1.74 mm
- net A6: track 69.7 -> 2.11 mm
- net A5: track 68.8 -> 2.01 mm
- net A4: track 68.7 -> 2.95 mm
- net A1: track 67.9 -> 2.29 mm
- net A3: track 67.9 -> 2.33 mm
- net A2: track 67.9 -> 2.33 mm
- net +5V: track 126.6 -> 93.9 mm
- net LED: track 67.0 -> 42.0 mm
- net Net-(U1-A02): track 25.2 -> 7.58 mm
- net Net-(U1-B02): track 26.3 -> 10.3 mm
- net SWITCH: track 51.1 -> 65.8 mm
- net Net-(J1-Pin_2): track 12.4 -> 25.5 mm, vias 0 -> 2
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- added copper zone on B.Cu, net GND
Other:
- board size 120 x 160 mm -> 120 x 123.9 mm

Commit message: act placa
Parts:
- moved J4 19.2 mm to (111.0, 90.7)
- moved Tornillo_M3_8mm 2.26 mm to (127.3, 90.5)
- moved Tornillo_M3_8mm 0.39 mm to (69.7, 90.5)
Routing:
- net +3.3V: track 7.68 -> 44.3 mm
- net A3: track 2.33 -> 15.3 mm
- net A4: track 2.95 -> 15.2 mm
- net A8: track 1.75 -> 13.0 mm
- net A7: track 1.74 -> 13.0 mm
- net A5: track 2.01 -> 13.0 mm
- net A6: track 2.11 -> 13.0 mm
- net A1: track 2.29 -> 12.9 mm
- net A2: track 2.33 -> 12.9 mm
- net GND: track 0.00 -> 7.90 mm, vias 0 -> 2
Other:
- board size 120 x 123.9 mm -> 120 x 106.2 mm
