File: hardware/velocista/velocista.kicad_pcb (KiCad board)
At the start: 2 copper layers, 120 x 106.2 mm, 19 parts, among them J1 XT30, J2 Cable_PAD, J3 Cable_PAD, J4 QTR8a, SW1 SW_Push, SW3 SW_SPDT, U1 TB6612FNG, U2 Mini360, U3 ESP32_DEVKITC

Commit message: act placa
Parts:
- moved D1 33.9 mm to (147.2, 92.6), turned to 0 degrees
- moved D2 33.1 mm to (73.3, 92.2), turned to 180 degrees
- moved R2 19.0 mm to (73.3, 85.3), turned to 90 degrees
- moved R1 19.0 mm to (147.2, 85.3), turned to -90 degrees
- moved J1 9.08 mm to (147.0, 77.4)
- moved SW1 5.05 mm to (73.3, 78.2)
- moved J3 4.01 mm to (116.0, 119.9)
- moved C1 4.01 mm to (117.7, 112.3)
- moved J2 3.47 mm to (98.5, 119.8)
- moved C2 3.47 mm to (102.9, 112.2)
Routing:
- net VCC: track 86.8 -> 54.8 mm
- net Net-(U1-A02): track 10.4 -> 30.3 mm
- net Net-(U1-A01): track 10.2 -> 26.2 mm
- net Net-(U1-B02): track 10.7 -> 26.0 mm
- net LED: track 42.0 -> 57.2 mm
- net SWITCH: track 67.0 -> 54.5 mm
- net Net-(U1-B01): track 9.56 -> 21.5 mm
- net Net-(J1-Pin_2): track 26.3 -> 34.0 mm, vias 2 -> 0
- net +3.3V: track 44.3 -> 45.7 mm
