File: hardware/velocista/velocista.kicad_pcb (KiCad board)
At the start: 2 copper layers, 120 x 106.2 mm, 19 parts, among them J1 XT30, J2 Cable_PAD, J3 Cable_PAD, J4 QTR8a, SW1 SW_Push, SW3 SW_SPDT, U1 TB6612FNG, U2 Mini360, U3 ESP32_DEVKITC

Commit message: act placa xd
Routing:
- net Net-(U1-B01): track 21.5 -> 22.8 mm
- net Net-(U1-A01): track 26.2 -> 27.3 mm
- net Net-(U1-B02): track 26.0 -> 26.6 mm
Changed lines of the file:
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@@
+	)
+	(segment
+		(start 118.79 111.33)
+		(end 121.2 113.74)
+		(width 1)
+		(layer "B.Cu")
+		(net 14)
+	)
+	(segment
+		(start 120.33 118.37)
+		(end 119.02 118.37)
+		(width 1)
+		(layer "B.Cu")
+		(net 14)
+	)
+	(segment
+		(start 117.72 109.52)
+		(end 116.644366 108.444366)
+		(width 1)
+		(layer "B.Cu")
+		(net 14)
+	)
+	(segment
+		(start 119.02 118.37)
+		(end 118.97 118.32)
+		(width 1)
+		(layer "B.Cu")
+		(net 14)
+	)
+	(segment
+		(start 121.2 113.74)
+		(end 121.2 117.5)
+		(width 1)
+		(layer "B.Cu")
+		(net 14)
+	)
+	(segment
+		(start 116.644366 108.444366)
+		(end 116.644366 99.836059)
+		(width 1)
+		(layer "B.Cu")
+		(net 14)
+	)
+	(segment
+		(start 121.2 117.5)
+		(end 120.33 118.37)
+		(width 1)
+		(layer "B.Cu")
+		(net 14)
+	)
+	(segment
+		(start 117.72 111.33)
+		(end 117.72 109.52)
+		(width 1)
+		(layer "B.Cu")
+		(net 14)
 	)
 	(segment
 		(start 117.72 111.33)
 		(end 118.79 111.33)
-		(width 1)
-		(layer "B.Cu")
-		(net 14)
-	)
-	(segment
-		(start 116.644366 110.254366)
-		(end 116.644366 99.836059)
-		(width 1)
-		(layer "B.Cu")
-		(net 14)
-	)
-	(segment
-		(start 119.02 118.37)
-		(end 118.97 118.32)
-		(width 1)
-		(layer "B.Cu")
-		(net 14)
-	)
-	(segment
-		(start 120.57 116.82)
-		(end 119.02 118.37)
-		(width 1)
-		(layer "B.Cu")
-		(net 14)
-	)
-	(segment
-		(start 117.72 111.33)
-		(end 116.644366 110.254366)
-		(width 1)
-		(layer "B.Cu")
-		(net 14)
-	)
-	(segment
-		(start 120.57 113.11)
-		(end 120.57 116.82)
-		(width 1)
-		(layer "B.Cu")
-		(net 14)
-	)
-	(segment
-		(start 118.79 111.33)
-		(end 120.57 113.11)
 		(width 1)
 		(layer "B.Cu")
@@
 	)
 	(segment
+		(start 114.104366 111.404366)
+		(end 114.104366 99.836059)
+		(width 1)
+		(layer "B.Cu")
+		(net 16)
+	)
+	(segment
+		(start 115.93 113.23)
+		(end 114.104366 111.404366)
+		(width 1)
+		(layer "B.Cu")
+		(net 16)
+	)
+	(segment
+		(start 116.25 120.06)
+		(end 117.36 121.17)
+		(width 1)
+		(layer "B.Cu")
+		(net 16)
+	)
+	(segment
+		(start 116.25 116.45)
+		(end 116.25 120.06)
+		(width 1)
+		(layer "B.Cu")
+		(net 16)
+	)
+	(segment
 		(start 117.36 121.17)
 		(end 119.02 121.17)
@@
 	(segment
 		(start 117.72 113.23)
-		(end 116.995 113.23)
-		(width 1)
-		(layer "B.Cu")
-		(net 16)
-	)
-	(segment
-		(start 116.25 120.06)
-		(end 117.36 121.17)
-		(width 1)
-		(layer "B.Cu")
-		(net 16)
-	)
-	(segment
-		(start 116.25 114.7)
-		(end 116.25 120.06)
-		(width 1)
-		(layer "B.Cu")
-		(net 16)
-	)
-	(segment
-		(start 114.104366 110.339366)
-		(end 114.104366 99.836059)
+		(end 117.72 114.98)
+		(width 1)
+		(layer "B.Cu")
+		(net 16)
+	)
+	(segment
+		(start 117.72 114.98)
+		(end 116.25 116.45)
 		(width 1)
 		(layer "B.Cu")
@@
 	(segment
 		(start 117.72 113.23)
-		(end 116.25 114.7)
-		(width 1)
-		(layer "B.Cu")
-		(net 16)
-	)
-	(segment
-		(start 116.995 113.23)
-		(end 114.104366 110.339366)
-		(width 1)
-		(layer "B.Cu")
-		(net 16)
+		(end 115.93 113.23)
+		(width 1)
+		(layer "B.Cu")
+		(net 16)
+	)
+	(segment
+		(start 104.225 116.325)
+		(end 104.225 119.83)
+		(width 1)
+		(layer "B.Cu")
+		(net 17)
 	)
 	(segment
 		(start 102.865 113.16)
-		(end 104.225 114.52)
-		(width 1)
-		(layer "B.Cu")
-		(net 17)
-	)
-	(segment
-		(start 104.225 114.52)
-		(end 104.225 119.83)
+		(end 107.93 113.16)
+		(width 1)
+		(layer "B.Cu")
+		(net 17)
+	)
+	(segment
+		(start 104.205 119.83)
+		(end 102.925 121.11)
+		(width 1)
+		(layer "B.Cu")
+		(net 17)
+	)
+	(segment
+		(start 102.865 114.965)
+		(end 104.225 116.325)
+		(width 1)
+		(layer "B.Cu")
+		(net 17)
+	)
+	(segment
+		(start 111.564366 109.525634)
+		(end 111.564366 99.836059)
 		(width 1)
 		(layer "B.Cu")
@@
 	)
 	(segment
-		(start 104.205 119.83)
-		(end 102.925 121.11)
-		(width 1)
-		(layer "B.Cu")
-		(net 17)
-	)
-	(segment
-		(start 102.865 113.16)
-		(end 107.93 113.16)
-		(width 1)
-		(layer "B.Cu")
-		(net 17)
-	)
-	(segment
-		(start 111.564366 109.525634)
-		(end 111.564366 99.836059)
-		(width 1)
-		(layer "B.Cu")
-		(net 17)
-	)
-	(segment
 		(start 102.925 121.11)
 		(end 101.55 121.11)
@@
 	)
 	(segment
+		(start 102.865 113.16)
+		(end 102.865 114.965)
+		(width 1)
+		(layer "B.Cu")
+		(net 17)
+	)
+	(segment
 		(start 101.404366 84.596059)
 		(end 101.404366 81.556059)
@@
 	(segment
 		(start 101.405 111.26)
-		(end 99.405 113.26)
+		(end 99 113.665)
+		(width 1)
+		(layer "B.Cu")
+		(net 19)
+	)
+	(segment
+		(start 100.21 118.31)
+		(end 101.55 118.31)
+		(width 1)
+		(layer "B.Cu")
+		(net 19)
+	)
+	(segment
+		(start 99 113.665)
+		(end 99 117.1)
 		(width 1)
 		(layer "B.Cu")
@@
 	)
 	(segment
+		(start 99 117.1)
+		(end 100.21 118.31)
+		(width 1)
+		(layer "B.Cu")
+		(net 19)
+	)
+	(segment
+		(start 109.024366 108.495634)
+		(end 109.024366 99.836059)
+		(width 1)
+		(layer "B.Cu")
+		(net 19)
+	)
+	(segment
 		(start 102.865 111.26)
 		(end 101.405 111.26)
 		(width 1)
 		(layer "B.Cu")
-		(net 19)
-	)
-	(segment
-		(start 109.024366 108.495634)
-		(end 109.024366 99.836059)
-		(width 1)
-		(layer "B.Cu")
-		(net 19)
-	)
-	(segment
-		(start 99.405 113.26)
-		(end 99.405 116.165)
-		(width 1)
-		(layer "B.Cu")
-		(net 19)
-	)
-	(segment
-		(start 99.405 116.165)
-		(end 101.55 118.31)
-		(width 1)
-		(layer "B.Cu")

Commit message: act placa
Routing:
- net +5V: track 93.9 -> 95.4 mm
- net LED: track 57.2 -> 58.0 mm
Changed lines of the file:
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@@
 	)
 	(segment
-		(start 98.714366 87.006059)
-		(end 96.324366 84.616059)
+		(start 98.714366 87.014366)
+		(end 98.714366 85.414366)
 		(width 1)
 		(layer "B.Cu")
@@
 	)
 	(segment
-		(start 98.714366 87.016059)
-		(end 98.714366 87.006059)
-		(width 1)
-		(layer "B.Cu")
-		(net 1)
-	)
-	(segment
 		(start 103.944366 99.246059)
 		(end 103.944366 99.836059)
@@
 	)
 	(segment
+		(start 98.714366 85.414366)
+		(end 97.916059 84.616059)
+		(width 1)
+		(layer "B.Cu")
+		(net 1)
+	)
+	(segment
 		(start 83.794366 53.736059)
 		(end 85.254366 52.276059)
@@
 	)
 	(segment
-		(start 99.834366 88.136059)
-		(end 98.714366 87.016059)
-		(width 1)
-		(layer "B.Cu")
-		(net 1)
-	)
-	(segment
 		(start 85.254366 52.276059)
 		(end 87.444366 52.276059)
@@
 	)
 	(segment
-		(start 109.024366 86.096059)
-		(end 106.984366 88.136059)
+		(start 97.916059 84.616059)
+		(end 96.324366 84.616059)
 		(width 1)
 		(layer "B.Cu")
@@
 	)
 	(segment
+		(start 109.024366 86.675634)
+		(end 107.2 88.5)
+		(width 1)
+		(layer "B.Cu")
+		(net 1)
+	)
+	(segment
 		(start 103.944366 99.836059)
 		(end 103.944366 99.106059)
@@
 	)
 	(segment
-		(start 106.984366 88.136059)
-		(end 99.834366 88.136059)
+		(start 107.2 88.5)
+		(end 100.2 88.5)
 		(width 1)
 		(layer "B.Cu")
@@
 	)
 	(segment
+		(start 100.2 88.5)
+		(end 98.714366 87.014366)
+		(width 1)
+		(layer "B.Cu")
+		(net 1)
+	)
+	(segment
 		(start 83.794366 76.096059)
 		(end 83.794366 53.736059)
@@
 	)
 	(segment
-		(start 109.024366 84.596059)
-		(end 109.024366 86.096059)
-		(width 1)
-		(layer "B.Cu")
-		(net 1)
-	)
-	(segment
 		(start 103.944366 99.836059)
 		(end 103.944366 102.846059)
+		(width 1)
+		(layer "B.Cu")
+		(net 1)
+	)
+	(segment
+		(start 109.024366 84.596059)
+		(end 109.024366 86.675634)
 		(width 1)
 		(layer "B.Cu")
@@
 	)
 	(segment
-		(start 97.8 42.465425)
-		(end 97.8 40.8)
+		(start 133.164366 47.464366)
+		(end 133.164366 52.276059)
 		(width 0.7)
 		(layer "B.Cu")
@@
 	)
 	(segment
-		(start 97.8 40.8)
-		(end 98.9 39.7)
+		(start 98.8 39.8)
+		(end 125.5 39.8)
 		(width 0.7)
 		(layer "B.Cu")
@@
 	)
 	(segment
-		(start 125.6 39.7)
-		(end 133.164366 47.264366)
-		(width 0.7)
-		(layer "B.Cu")
-		(net 10)
-	)
-	(segment
-		(start 98.9 39.7)
-		(end 125.6 39.7)
-		(width 0.7)
-		(layer "B.Cu")
-		(net 10)
-	)
-	(segment
-		(start 133.164366 47.264366)
-		(end 133.164366 52.276059)
-		(width 0.7)
-		(layer "B.Cu")
-		(net 10)
-	)
-	(segment
-		(start 81.864366 78.435634)
-		(end 76.02 84.28)
-		(width 1)
-		(layer "B.Cu")
-		(net 11)
-	)
-	(segment
-		(start 76.02 84.28)
+		(start 97.794366 40.805634)
+		(end 98.8 39.8)
+		(width 0.7)
+		(layer "B.Cu")
+		(net 10)
+	)
+	(segment
+		(start 125.5 39.8)
+		(end 133.164366 47.464366)
+		(width 0.7)
+		(layer "B.Cu")
+		(net 10)
+	)
+	(segment
+		(start 97.794366 42.471059)
+		(end 97.794366 40.805634)
+		(width 0.7)
+		(layer "B.Cu")
+		(net 10)
+	)
+	(segment
+		(start 81.864366 52.616059)
+		(end 81.864366 81.035634)
+		(width 1)
+		(layer "B.Cu")
+		(net 11)
+	)
+	(segment
+		(start 97.604366 52.276059)
+		(end 97.604366 50.504366)
+		(width 1)
+		(layer "B.Cu")
+		(net 11)
+	)
+	(segment
+		(start 81.864366 81.035634)
+		(end 78.62 84.28)
+		(width 1)
+		(layer "B.Cu")
+		(net 11)
+	)
+	(segment
+		(start 78.62 84.28)
 		(end 73.31 84.28)
 		(width 1)
@@
 	)
 	(segment
-		(start 97.604366 52.276059)
-		(end 97.604366 49.746059)
-		(width 1)
-		(layer "B.Cu")
-		(net 11)
-	)
-	(segment
-		(start 81.864366 52.616059)
-		(end 81.864366 78.435634)
-		(width 1)
-		(layer "B.Cu")
-		(net 11)
-	)
-	(segment
-		(start 96.444366 48.586059)
-		(end 85.894366 48.586059)
-		(width 1)
-		(layer "B.Cu")
-		(net 11)
-	)
-	(segment
-		(start 97.604366 49.746059)
-		(end 96.444366 48.586059)
-		(width 1)
-		(layer "B.Cu")
-		(net 11)
-	)
-	(segment
-		(start 85.894366 48.586059)
+		(start 97.604366 50.504366)
+		(end 96 48.9)
+		(width 1)
+		(layer "B.Cu")
+		(net 11)
+	)
+	(segment
+		(start 96 48.9)
+		(end 85.580425 48.9)
+		(width 1)
+		(layer "B.Cu")
+		(net 11)
+	)
+	(segment
+		(start 85.580425 48.9)
 		(end 81.864366 52.616059)
 		(width 1)

Commit message: act pcb
Parts:
- moved C2 8.18 mm to (110.2, 108.6), turned to 0 degrees
- moved J3 4.81 mm to (120.8, 119.8)
- moved C1 4.40 mm to (115.3, 108.6), turned to 0 degrees
Routing:
- net Net-(U1-A01): track 27.3 -> 23.4 mm
- net Net-(U1-A02): track 30.3 -> 26.9 mm
- net Net-(U1-B01): track 22.8 -> 23.6 mm

Commit message: act pcb
Parts:
- removed U3: ESP32_DEVKITC, EESTN5:ESP32S
- added U4: ESP32-DEVKITC-32D, a:MODULE_ESP32-DEVKITC-32D, F.Cu at (112.2, 66.1)
Routing:
- net BM2: track 10.6 -> 5.83 mm
- net AM1: track 10.4 -> 5.83 mm
- net PWM2: track 11.3 -> 6.88 mm
- net BM1: track 10.0 -> 5.83 mm
- net AM2: track 9.99 -> 5.83 mm
- net PWM1: track 9.99 -> 5.83 mm
- net LED: track 58.0 -> 55.1 mm
- net +3.3V: track 45.5 -> 47.8 mm
- net A8: track 13.0 -> 14.3 mm
- net A6: track 13.0 -> 14.1 mm
- net A3: track 12.9 -> 14.1 mm
- net A2: track 12.9 -> 14.1 mm
- net A7: track 13.0 -> 14.1 mm
- net A5: track 13.0 -> 14.1 mm
- net A4: track 12.9 -> 14.0 mm
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
Commit message: actu pcb
Routing:
- net GND: track 7.60 -> 6.70 mm
- net SWITCH: track 54.5 -> 54.0 mm
Changed lines of the file:
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@@
 	)
 	(segment
-		(start 130.3 47.5)
-		(end 130.3 39.9)
+		(start 128.4 47.5)
+		(end 135.1 47.5)
 		(width 1)
 		(layer "F.Cu")
@@
 	)
 	(via
-		(at 130.3 39.9)
+		(at 135.1 47.5)
 		(size 1.25)
 		(drill 0.75)
@@
 	)
 	(via
-		(at 130.3 47.5)
+		(at 128.4 47.5)
 		(size 1.25)
 		(drill 0.75)
@@
 	)
 	(segment
-		(start 110.294366 42.471059)
-		(end 110.294366 43.844366)
-		(width 0.7)
+		(start 110.294366 44.394366)
+		(end 110.294366 42.471059)
+		(width 1)
 		(layer "B.Cu")
 		(net 9)
 	)
 	(segment
-		(start 110.294366 43.844366)
-		(end 116.72 50.27)
-		(width 0.7)
+		(start 116.72 50.82)
+		(end 110.294366 44.394366)
+		(width 1)
 		(layer "B.Cu")
 		(net 9)
 	)
 	(segment
-		(start 116.72 50.27)
-		(end 116.72 53.4)
-		(width 0.7)
+		(start 116.72 53.4)
+		(end 116.72 50.82)
+		(width 1)
 		(layer "B.Cu")
 		(net 9)
@@
 	)
 	(segment
+		(start 104 53.38)
+		(end 104 51.5)
+		(width 1)
+		(layer "B.Cu")
+		(net 12)
+	)
+	(segment
+		(start 73.3 56.4)
+		(end 73.3 71.65)
+		(width 1)
+		(layer "B.Cu")
+		(net 12)
+	)
+	(segment
 		(start 83.103941 46.596059)
 		(end 73.3 56.4)
@@
 	)
 	(segment
-		(start 104 50.55)
-		(end 100.046059 46.596059)
-		(width 1)
-		(layer "B.Cu")
-		(net 12)
-	)
-	(segment
-		(start 73.3 56.4)
-		(end 73.3 71.65)
-		(width 1)
-		(layer "B.Cu")
-		(net 12)
-	)
-	(segment
-		(start 104 53.38)
-		(end 104 50.55)
-		(width 1)
-		(layer "B.Cu")
-		(net 12)
-	)
-	(segment
 		(start 104.02 53.4)
 		(end 104 53.38)
@@
 	)
 	(segment
-		(start 100.046059 46.596059)
+		(start 99.096059 46.596059)
 		(end 83.103941 46.596059)
 		(width 1)
 		(layer "B.Cu")
 		(net 12)
+	)
+	(segment
+		(start 104 51.5)
+		(end 99.096059 46.596059)
+		(width 1)
+		(layer "B.Cu")
+		(net 12)
+	)
+	(segment
+		(start 119.26 50.91)
+		(end 112.794366 44.444366)
+		(width 1)
+		(layer "B.Cu")
+		(net 13)
+	)
+	(segment
+		(start 112.794366 44.444366)
+		(end 112.794366 42.471059)
+		(width 1)
+		(layer "B.Cu")
+		(net 13)
 	)
 	(segment
@@
 	)
 	(segment
-		(start 119.26 50.36)
-		(end 119.26 53.4)
-		(width 0.7)
-		(layer "B.Cu")
-		(net 13)
-	)
-	(segment
-		(start 112.794366 43.894366)
-		(end 119.26 50.36)
-		(width 0.7)
-		(layer "B.Cu")
-		(net 13)
-	)
-	(segment
-		(start 112.794366 42.471059)
-		(end 112.794366 43.894366)
-		(width 0.7)
+		(start 119.26 53.4)
+		(end 119.26 50.91)
+		(width 1)
 		(layer "B.Cu")
 		(net 13)
@@
 	)
 	(segment
-		(start 115.294366 43.894366)
-		(end 121.8 50.4)
-		(width 0.7)
+		(start 121.8 53.4)
+		(end 121.8 50.75)
+		(width 1)
 		(layer "B.Cu")
 		(net 20)
 	)
 	(segment
-		(start 121.8 50.4)
-		(end 121.8 53.4)
-		(width 0.7)
-		(layer "B.Cu")
-		(net 20)
-	)
-	(segment
-		(start 115.294366 42.471059)
-		(end 115.294366 43.894366)
-		(width 0.7)
+		(start 121.8 50.75)
+		(end 115.294366 44.244366)
+		(width 1)
 		(layer "B.Cu")
 		(net 20)
@@
 	)
 	(segment
-		(start 100.294366 44.144366)
-		(end 106.56 50.41)
-		(width 0.7)
+		(start 115.294366 44.244366)
+		(end 115.294366 42.471059)
+		(width 1)
+		(layer "B.Cu")
+		(net 20)
+	)
+	(segment
+		(start 100.294366 44.994366)
+		(end 100.294366 42.471059)
+		(width 1)
 		(layer "B.Cu")
 		(net 21)
 	)
 	(segment
-		(start 106.56 50.41)
-		(end 106.56 53.4)
-		(width 0.7)
+		(start 106.56 53.4)
+		(end 106.56 51.26)
+		(width 1)
+		(layer "B.Cu")
+		(net 21)
+	)
+	(segment
+		(start 106.56 51.26)
+		(end 100.294366 44.994366)
+		(width 1)
 		(layer "B.Cu")
 		(net 21)
@@
 	)
 	(segment
-		(start 100.294366 42.471059)
-		(end 100.294366 44.144366)
-		(width 0.7)
-		(layer "B.Cu")
-		(net 21)
-	)
-	(segment
-		(start 102.794366 44.244366)
-		(end 109.1 50.55)
-		(width 0.7)
+		(start 109.1 51)
+		(end 102.794366 44.694366)
+		(width 1)
 		(layer "B.Cu")
 		(net 22)
 	)
 	(segment
-		(start 109.1 50.55)
-		(end 109.1 53.4)
-		(width 0.7)
+		(start 102.794366 44.694366)
+		(end 102.794366 42.471059)
+		(width 1)
 		(layer "B.Cu")
 		(net 22)
@@
 	)
 	(segment
-		(start 102.794366 42.471059)
-		(end 102.794366 44.244366)
-		(width 0.7)
+		(start 109.1 53.4)
+		(end 109.1 51)
+		(width 1)
 		(layer "B.Cu")
 		(net 22)
 	)
 	(segment
-		(start 117.794366 42.471059)
-		(end 117.794366 44.069366)
-		(width 0.7)
+		(start 124.34 53.4)
+		(end 124.34 50.54)
+		(width 1)
 		(layer "B.Cu")
 		(net 23)
 	)
 	(segment
-		(start 117.794366 44.069366)
-		(end 124.34 50.615)
-		(width 0.7)
+		(start 117.794366 43.994366)
+		(end 117.794366 42.471059)
+		(width 1)
 		(layer "B.Cu")
 		(net 23)
@@
 	)
 	(segment
-		(start 124.34 50.615)
-		(end 124.34 53.4)
-		(width 0.7)
+		(start 124.34 50.54)
+		(end 117.794366 43.994366)
+		(width 1)
 		(layer "B.Cu")
 		(net 23)
 	)
 	(segment
-		(start 114.18 50.48)
-		(end 114.18 53.4)
-		(width 0.7)
+		(start 114.18 50.88)
+		(end 107.794366 44.494366)
+		(width 1)
 		(layer "B.Cu")
 		(net 24)
 	)
 	(segment
-		(start 107.794366 44.094366)
-		(end 114.18 50.48)
-		(width 0.7)
+		(start 114.18 53.4)
+		(end 114.18 50.88)
+		(width 1)
 		(layer "B.Cu")
 		(net 24)
 	)
 	(segment
-		(start 107.794366 42.471059)
-		(end 107.794366 44.094366)
-		(width 0.7)
+		(start 107.794366 44.494366)
+		(end 107.794366 42.471059)
+		(width 1)
 		(layer "B.Cu")
 		(net 24)
@@
 	)
 	(segment
-		(start 105.294366 44.194366)
-		(end 111.64 50.54)
-		(width 0.7)
+		(start 111.64 50.84)
+		(end 105.294366 44.494366)
+		(width 1)
 		(layer "B.Cu")
 		(net 25)
 	)
 	(segment
-		(start 105.294366 42.471059)
-		(end 105.294366 44.194366)
-		(width 0.7)
+		(start 111.64 53.4)
+		(end 111.64 50.84)
+		(width 1)
 		(layer "B.Cu")
 		(net 25)
@@
 	)
 	(segment
-		(start 111.64 50.54)
-		(end 111.64 53.4)
-		(width 0.7)
+		(start 105.294366 44.494366)
+		(end 105.294366 42.471059)
+		(width 1)
 		(layer "B.Cu")
 		(net 25)
